Commit message: feat(fa): 新增可选视觉标定位姿发布并更新关节限位 - 新增 /sysmo_vision_calibration 位姿发布，支持选择左右手和配置频率 - 标定默认关闭，仅在发布频率大于零时加载消息依赖、创建发布器并执行标定计算 - 同步更新 FA 控制配置与 URDF 中的双臂及颈部关节限位 - 调整测试以匹配 min-snap 路由、局部逃逸、状态新鲜度检查和多 seed IK 策略
验证：FA 适配测试 53 项通过，git diff --check 通过；未进行实机验证

File: beavr-bot/robots/fa_description/urdf/fa_robot.urdf (robot description, URDF)
Before this commit: robot fa_robot, 56 links, 55 joints
Joints:
- joint left_elbow_joint: limit lower=-1.4 upper=0.26 effort=0 velocity=0 -> lower=-2.050 upper=1.440 effort=0 velocity=0
- joint left_shoulder_pitch_joint: limit lower=-2.79 upper=2.79 effort=0 velocity=0 -> lower=-2.750 upper=2.748 effort=0 velocity=0
- joint left_shoulder_roll_joint: limit lower=-0.33 upper=3.49 effort=0 velocity=0 -> lower=-0.288 upper=3.342 effort=0 velocity=0
- joint left_shoulder_yaw_joint: limit lower=-2.79 upper=2.79 effort=0 velocity=0 -> lower=-2.650 upper=2.583 effort=0 velocity=0
- joint left_wrist_pitch_joint: limit lower=-0.52 upper=0.52 effort=0 velocity=0 -> lower=-0.469 upper=0.482 effort=0 velocity=0
- joint left_wrist_roll_joint: limit lower=-1.57 upper=1.57 effort=0 velocity=0 -> lower=-1.550 upper=1.520 effort=0 velocity=0
- joint left_wrist_yaw_joint: limit lower=-2.79 upper=2.79 effort=0 velocity=0 -> lower=-2.735 upper=2.729 effort=0 velocity=0
- joint neck_pitch_joint: limit lower=-0.52 upper=0.79 effort=0 velocity=0 -> lower=-0.523 upper=0.785 effort=0 velocity=0
- joint neck_yaw_joint: limit lower=-1.57 upper=1.57 effort=0 velocity=0 -> lower=-1.570 upper=1.570 effort=0 velocity=0
- joint right_elbow_joint: limit lower=-1.4 upper=0.26 effort=0 velocity=0 -> lower=-2.050 upper=1.440 effort=0 velocity=0
- joint right_shoulder_pitch_joint: limit lower=-2.79 upper=2.79 effort=0 velocity=0 -> lower=-2.750 upper=2.750 effort=0 velocity=0
- joint right_shoulder_roll_joint: limit lower=-3.49 upper=0.33 effort=0 velocity=0 -> lower=-3.330 upper=0.302 effort=0 velocity=0
- joint right_shoulder_yaw_joint: limit lower=-2.79 upper=2.79 effort=0 velocity=0 -> lower=-2.570 upper=2.660 effort=0 velocity=0
- joint right_wrist_pitch_joint: limit lower=-0.52 upper=0.52 effort=0 velocity=0 -> lower=-0.480 upper=0.470 effort=0 velocity=0
- joint right_wrist_roll_joint: limit lower=-1.57 upper=1.57 effort=0 velocity=0 -> lower=-1.536 upper=1.532 effort=0 velocity=0
- joint right_wrist_yaw_joint: limit lower=-2.79 upper=2.79 effort=0 velocity=0 -> lower=-2.730 upper=2.730 effort=0 velocity=0
